Commit message: bugfix von angle funktion

File: common/roslisp_common/cl_urdf/test_urdfs/pr2.urdf (robot description, URDF)
Before this commit: robot pr2, 81 links, 80 joints
Joints:
- joint torso_lift_joint: limit lower=0.0 upper=0.31 effort=10000 velocity=0.013 -> lower=0.0 upper=1.2 effort=10000 velocity=0.013; origin xyz=-0.05 0 0.739675 rpy=0 0 0 -> xyz=-0.05 0 1.2 rpy=0 0 0
